File: Hardware/Plantomation.kicad_pcb (KiCad board)
At the start: 2 copper layers, 100 x 80 mm, 91 parts, among them J1 12V, J11 Valve 3, J12 Valve 4, J13 Ch_Sel, J14 SD_Card, J2 USB_B, J3 ADC1_4, J4 ADC1_5, J5 ADC1_6, J6 ADC1_7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

Commit message: Finishing Touches on Layout before Review
Parts:
- added C20: 1n, Capacitor_SMD:C_0805_2012Metric, F.Cu at (164.6, 82.8)
- added HS1: D²PAK, Heatsink:Heatsink_Fischer_FK24413DPAK_23x13mm, F.Cu at (107.4, 106.9)
- added J10: ADC1_0, Connector_JST:JST_XH_B2B-XH-A_1x02_P2.50mm_Vertical, F.Cu at (158.5, 78.8)
- added R28: 100, Resistor_SMD:R_0805_2012Metric, F.Cu at (162.6, 82.8)
- added R29: 10k, Resistor_SMD:R_0805_2012Metric, F.Cu at (166.6, 82.8)
- added R30: 1k, Resistor_SMD:R_0805_2012Metric, F.Cu at (174.8, 114.6)
- C15, C16, C17, C18: value 100n -> 1n
- J14: value SD_Card -> GSD090012SEU
- JP1: value Jumper_2_Open -> VBUS Jumper
- moved C10 4.06 mm to (121.4, 105.2)
- moved C8 4.06 mm to (121.4, 108.7)
- moved C7 4.06 mm to (119.4, 108.7)
- moved C9 4.06 mm to (119.4, 105.2)
- moved REF** 3.09 mm to (169.9, 94.5)
- moved G*** 3.05 mm to (155.4, 91.7)
- moved REF** 0.51 mm to (169.7, 107.4)
- moved REF** 0.51 mm to (155.4, 107.4)
Connections:
- net Ch1_LedOK renamed Ch1_Led
- net Ch2_LedOK renamed Ch2_Led
- net Ch3_LedOK renamed Ch3_Led
- net Ch4_LedOK renamed Ch4_Led
- net EN renamed ~{EN}
- net /Detect renamed ~{Detect}
- net /Protect renamed ~{Protect}
- U1 pad 4: unconnected-(U1-SENSOR_VP-Pad4) -> Spill
- U5 pad 9: unconnected-(U5-~{RST}-Pad9) -> Net-(U5-~{RST})
Routing:
- net Spill: track 0.00 -> 60.6 mm, vias 0 -> 4
- net Net-(U5-VDD): track 2.01 -> 12.3 mm, vias 0 -> 2
- net Net-(U5-~{RST}): track 0.00 -> 9.63 mm, vias 0 -> 2
- net +12V: track 82.7 -> 87.6 mm
- net Net-(J10-Pin_2): track 0.00 -> 4.31 mm
- net GND: track 55.4 -> 59.0 mm, vias 209 -> 74
- net +3V3: track 157.6 -> 159.9 mm
- net +5V: track 173.1 -> 174.7 mm
- net SD0: track 37.8 -> 37.2 mm
- net ~{EN}: track 104.9 -> 105.4 mm
Other:
- board text added: "Spill"

Commit message: Big Repo Overhaul Started Documentation First Review Overhaul of Schematic and Layout First working Test Code for webpage and OTA
Parts:
- removed J13: Ch_Sel, Connector_PinHeader_2.54mm:PinHeader_2x02_P2.54mm_Vertical
- removed R26, R27: 1k, Resistor_SMD:R_0805_2012Metric
- added R31: 4k7, Resistor_SMD:R_0805_2012Metric, F.Cu at (133.1, 98.3)
- R11, R4: value 100 -> 4k7
- moved J5 84.2 mm to (115.6, 137.6), turned to 90 degrees
- moved J1 83.5 mm to (187.4, 136.3), turned to 180 degrees
- moved J6 77.9 mm to (123.7, 137.6), turned to 90 degrees
- moved D5 76.7 mm to (186.2, 131.1), turned to 180 degrees
- moved J7 73.7 mm to (187.4, 127.0), turned to 180 degrees
- moved J3 72.9 mm to (131.8, 137.6), turned to 90 degrees
- moved C1 70.7 mm to (113.5, 122.9), turned to 180 degrees
- moved J4 69.4 mm to (139.9, 137.6), turned to 90 degrees
- moved R1 68.9 mm to (113.5, 120.9), turned to 0 degrees
- moved H2 67.6 mm to (168.9, 45.5), turned to 90 degrees
- moved C3 66.6 mm to (113.5, 118.4), turned to 180 degrees
- moved HS1 66.2 mm to (168.1, 133.3), turned to 180 degrees
- moved D6 65.9 mm to (186.2, 120.4), turned to 180 degrees
- moved U3 65.8 mm to (168.1, 133.1), turned to -90 degrees
- moved C2 64.9 mm to (113.5, 116.3), turned to 180 degrees
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Connections:
- net Net-(U1-IO32) renamed /Sensor3
- net Net-(U1-IO33) renamed /Sensor4
- net Net-(U1-IO34) renamed /Sensor1
- net Net-(U1-IO35) renamed /Sensor2
- net PeriPump renamed Pump
- J14 pad 1: SD3 -> VSPI_CS
- J14 pad 2: CMD -> VSPI_MOSI
- J14 pad 5: CLK -> VSPI_CLK
- J14 pad 7: SD0 -> VSPI_MISO
- J14 pad 8: SD1 -> unconnected-(J14-DAT1-Pad8)
- J14 pad 9: SD2 -> unconnected-(J14-DAT2-Pad9)
- U1 pad 13: Net-(J13-Pin_1) -> ~{Protect}
- U1 pad 16: Net-(J13-Pin_3) -> ~{Detect}
- U1 pad 17: SD2 -> unconnected-(U1-SHD/SD2-Pad17)
- U1 pad 18: SD3 -> unconnected-(U1-SWP/SD3-Pad18)
- U1 pad 19: CMD -> unconnected-(U1-SCS/CMD-Pad19)
- U1 pad 20: CLK -> unconnected-(U1-SCK/CLK-Pad20)
- U1 pad 21: SD0 -> unconnected-(U1-SDO/SD0-Pad21)
- U1 pad 22: SD1 -> unconnected-(U1-SDI/SD1-Pad22)
- U1 pad 23: unconnected-(U1-IO15-Pad23) -> Ch4_Led
- U1 pad 24: unconnected-(U1-IO2-Pad24) -> Net-(U1-IO2)
- U1 pad 27: ~{Detect} -> Ch3_Led
- U1 pad 28: ~{Protect} -> Ch2_Led
- U1 pad 29: unconnected-(U1-IO5-Pad29) -> VSPI_CS
- U1 pad 30: Ch4_Led -> VSPI_CLK
- U1 pad 31: Ch3_Led -> VSPI_MISO
- U1 pad 33: Ch2_Led -> Ch1_Led
- U1 pad 36: Ch1_Led -> VSPI_MOSI
Routing:
- net Net-(J13-Pin_1): track 87.2 -> 0.00 mm, vias 2 -> 0
- net Net-(J13-Pin_3): track 83.1 -> 0.00 mm, vias 4 -> 0
- net SD2: track 46.4 -> 0.00 mm, vias 2 -> 0
- net SD3: track 44.2 -> 0.00 mm, vias 2 -> 0
- net CMD: track 41.9 -> 0.00 mm, vias 2 -> 0
- net CLK: track 40.4 -> 0.00 mm, vias 2 -> 0
- net SD1: track 37.5 -> 0.00 mm, vias 2 -> 0
- net SD0: track 37.2 -> 0.00 mm, vias 2 -> 0
- net VSPI_MISO: track 0.00 -> 34.2 mm, vias 0 -> 2
- net VSPI_CS: track 0.00 -> 31.9 mm, vias 0 -> 2
- net VSPI_MOSI: track 0.00 -> 31.7 mm, vias 0 -> 2
- net VSPI_CLK: track 0.00 -> 31.7 mm, vias 0 -> 2
- net ~{Protect}: track 43.2 -> 55.8 mm
- net Ch4_Led: track 6.58 -> 18.5 mm, vias 0 -> 2
- net ~{Detect}: track 38.4 -> 47.0 mm
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Other:
- board size 100 x 80 mm -> 80 x 100 mm
- board text added: "IP:"
- board text added: "SN:"
- board text removed: "1 2 3 4"
- board text removed: "No. of Channels"

Commit message: Finalizing PCB and Review Firmware Bugfixes for Ajax Firmware get a working responsive page layout
Parts:
- added G***: LOGO, TheBrutzlers_Lib:approved_theBrutzler, F.Cu at (154.4, 55.9)
- moved REF** 0.40 mm to (167.2, 68.8)
Connections:
- U2 pad 1: /Dp -> /Dm
- U2 pad 3: /Dm -> /Dp
- U2 pad 4: Net-(J2-D-) -> Net-(J2-D+)
- U2 pad 6: Net-(J2-D+) -> Net-(J2-D-)
Routing:
- net Pump: track 57.0 -> 51.6 mm
- net ~{EN}: track 105.4 -> 110.5 mm
- net /Dp: track 4.33 -> 8.92 mm
- net Ch4_Led: track 18.5 -> 14.7 mm
- net Valve 1: track 67.0 -> 63.6 mm
- net Valve 4: track 51.5 -> 54.8 mm
- net Net-(J2-D-): track 3.75 -> 6.53 mm
- net Net-(D4-A): track 0.00 -> 1.71 mm
- net Net-(D3-A): track 0.00 -> 1.71 mm
- net Net-(D2-A): track 0.00 -> 1.71 mm
- net Net-(D1-A): track 0.00 -> 1.71 mm
- net Valve 3: track 50.7 -> 52.4 mm
- net VSPI_MOSI: track 31.7 -> 33.3 mm
- net Net-(J2-D+): track 8.66 -> 7.77 mm
- net +5V: track 174.7 -> 175.3 mm
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