File: Hardware/Plantomation.kicad_sch (KiCad schematic)
At the start: 86 parts, among them J1 12V, J11 Valve 3, J12 Valve 4, J13 Ch_Sel, J14 GSD090012SEU, J2 USB_B, J3 ADC1_4, J4 ADC1_5, J5 ADC1_6, J6 ADC1_7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

Commit message: Finishing Touches on Layout before Review
Parts:
- added C20: 1n, Capacitor_SMD:C_0805_2012Metric, symbol Device:C
- added HS1: D²PAK, Heatsink:Heatsink_Fischer_FK24413DPAK_23x13mm, symbol Mechanical:Heatsink_Pad
- added J10: ADC1_0, Connector_JST:JST_XH_B2B-XH-A_1x02_P2.50mm_Vertical, symbol Connector_Generic:Conn_01x02
- added R28: 100, Resistor_SMD:R_0805_2012Metric, symbol Device:R
- added R29: 10k, Resistor_SMD:R_0805_2012Metric, symbol Device:R
- added R30: 1k, Resistor_SMD:R_0805_2012Metric, symbol Device:R
- C15, C16, C17, C18: value 100n -> 1n
- JP1: value Jumper_2_Open -> VBUS Jumper
Connections:
- net +3V3: now also J10.1 (Pin_1)
- net GND: now also C20.2, HS1.1, R29.2
- net at C19.1, U5.6 (VDD): now also R30.1
- net at U5.9 (~{RST}): now also R30.2
- net Spill: now reaches U1.4 (SENSOR_VP)
- net Spill: now also C20.1, R28.2, R29.1
- net Ch1_LedOK renamed Ch1_Led
- net Ch2_LedOK renamed Ch2_Led
- net Ch3_LedOK renamed Ch3_Led
- net Ch4_LedOK renamed Ch4_Led
- net EN renamed ~{EN}
- net /Detect renamed ~{Detect}
- net /Protect renamed ~{Protect}
- new net: J10.2 (Pin_2), R28.1
- no-connect marks 23 -> 21
Other:
- note added: "12V 3A Input"
- note added: "12V Pump"
- note added: "Spill Sensor"
- note removed: "Peristaltic Pump"
- moved on the sheet: C19, C4, C5, C6, D1, D2, D3, D4, FB1, J14, J3, J4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

Commit message: codebase and first part review
Parts:
- removed J13: Ch_Sel, Connector_PinHeader_2.54mm:PinHeader_2x02_P2.54mm_Vertical, symbol Connector_Generic:Conn_02x02_Odd_Even
- removed R26, R27: 1k, Resistor_SMD:R_0805_2012Metric, symbol Device:R
- added R31: 4k7, Resistor_SMD:R_0805_2012Metric, symbol Device:R
- R11, R4: value 100 -> 4k7
Connections:
- net Ch1_Led: now also U1.33 (IO21); no longer U1.36 (IO22)
- net Ch2_Led: now also U1.28 (IO17); no longer U1.33 (IO21)
- net Ch3_Led: now also U1.27 (IO16); no longer U1.31 (IO19)
- net Ch4_Led: now also U1.23 (IO15); no longer U1.30 (IO18)
- net GND: now also R31.2
- net ~{Detect}: now also U1.16 (IO13); no longer U1.27 (IO16)
- net ~{Protect}: now also U1.13 (IO14); no longer U1.28 (IO17)
- net at U1.24 (IO2): now also R31.1
- net VSPI_CS: now reaches U1.29 (IO5)
- net VSPI_CS: now also J14.1 (CD/DAT3)
- net CLK: no longer names the net of U1.20 (SCK/CLK)
- net CLK: no longer J14.5 (CLK)
- net CMD: no longer names the net of U1.19 (SCS/CMD)
- net CMD: no longer J14.2 (CMD)
- net PeriPump renamed Pump
- net SD0: no longer names the net of U1.21 (SDO/SD0)
- net SD0: no longer J14.7 (DAT0)
- net SD1: no longer names the net of J14.8 (DAT1)
- net SD1: no longer U1.22 (SDI/SD1)
- net SD2: no longer names the net of J14.9 (DAT2)
- net SD2: no longer U1.17 (SHD/SD2)
- net SD3: no longer names the net of U1.18 (SWP/SD3)
- net SD3: no longer J14.1 (CD/DAT3)
- new net VSPI_CLK: J14.5 (CLK), U1.30 (IO18)
- new net VSPI_MISO: J14.7 (DAT0), U1.31 (IO19)
- new net VSPI_MOSI: J14.2 (CMD), U1.36 (IO22)
- no-connect marks 21 -> 26

Commit message: Big Repo Overhaul Started Documentation First Review Overhaul of Schematic and Layout First working Test Code for webpage and OTA
Connections:
- net Sensor2: now reaches C18.1, R25.1, U1.7 (IO35)
- net Sensor3: now reaches C15.1, R22.1, U1.8 (IO32)
- net Sensor1: now reaches C17.1, R24.1, U1.6 (IO34)
- net Sensor4: now reaches C16.1, R23.1, U1.9 (IO33)
Other:
- note removed: "B08CZRLT7D"

Commit message: Finalizing PCB and Review Firmware Bugfixes for Ajax Firmware get a working responsive page layout
Connections:
- net Dm: now also U2.1 (I/O1); no longer U2.3 (I/O2)
- net Dp: now also U2.3 (I/O2); no longer U2.1 (I/O1)
- net at U2.4 (I/O2): now also J2.3 (D+); no longer J2.2 (D-)
- net at U2.6 (I/O1): now also J2.2 (D-); no longer J2.3 (D+)
Changed lines of the file:
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@@
     (stroke (width 0) (type default))
   )
-  (wire (pts (xy 59.69 147.955) (xy 59.69 144.145))
-    (stroke (width 0) (type default))
-  )
   (wire (pts (xy 92.71 101.6) (xy 92.71 100.33))
     (stroke (width 0) (type default))
@@
     (stroke (width 0) (type default))
   )
+  (wire (pts (xy 34.29 154.94) (xy 34.29 144.145))
+    (stroke (width 0) (type default))
+  )
   (wire (pts (xy 273.685 19.685) (xy 273.685 22.225))
     (stroke (width 0) (type default))
@@
     (stroke (width 0) (type default))
   )
-  (wire (pts (xy 78.74 150.495) (xy 78.74 168.91))
-    (stroke (width 0) (type default))
-  )
   (wire (pts (xy 209.55 85.09) (xy 209.55 87.63))
     (stroke (width 0) (type default))
@@
     (stroke (width 0) (type default))
   )
-  (wire (pts (xy 86.36 150.495) (xy 78.74 150.495))
+  (wire (pts (xy 73.025 150.495) (xy 86.36 150.495))
     (stroke (width 0) (type default))
   )
@@
     (stroke (width 0) (type default))
   )
+  (wire (pts (xy 74.295 168.91) (xy 53.34 168.91))
+    (stroke (width 0) (type default))
+  )
   (wire (pts (xy 185.42 95.25) (xy 185.42 99.06))
     (stroke (width 0) (type default))
@@
     (stroke (width 0) (type default))
   )
+  (wire (pts (xy 73.025 150.495) (xy 73.025 144.145))
+    (stroke (width 0) (type default))
+  )
   (wire (pts (xy 116.84 88.265) (xy 119.38 88.265))
     (stroke (width 0) (type default))
@@
     (stroke (width 0) (type default))
   )
-  (wire (pts (xy 78.74 168.91) (xy 53.34 168.91))
-    (stroke (width 0) (type default))
-  )
   (wire (pts (xy 154.94 88.9) (xy 154.94 93.98))
     (stroke (width 0) (type default))
@@
     (stroke (width 0) (type default))
   )
-  (wire (pts (xy 36.195 157.48) (xy 36.195 144.145))
-    (stroke (width 0) (type default))
-  )
   (wire (pts (xy 218.44 76.2) (xy 218.44 86.36))
     (stroke (width 0) (type default))
@@
     (stroke (width 0) (type default))
   )
+  (wire (pts (xy 36.195 168.91) (xy 48.26 168.91))
+    (stroke (width 0) (type default))
+  )
   (wire (pts (xy 31.75 149.86) (xy 31.75 127))
     (stroke (width 0) (type default))
@@
     (stroke (width 0) (type default))
   )
-  (wire (pts (xy 86.36 147.955) (xy 59.69 147.955))
-    (stroke (width 0) (type default))
-  )
   (wire (pts (xy 17.78 38.1) (xy 16.51 38.1))
     (stroke (width 0) (type default))
@@
     (stroke (width 0) (type default))
   )
-  (wire (pts (xy 59.69 144.145) (xy 53.34 144.145))
+  (wire (pts (xy 74.295 147.955) (xy 74.295 168.91))
     (stroke (width 0) (type default))
   )
@@
     (stroke (width 0) (type default))
   )
+  (wire (pts (xy 53.34 144.145) (xy 73.025 144.145))
+    (stroke (width 0) (type default))
+  )
   (wire (pts (xy 116.84 88.265) (xy 116.84 80.01))
     (stroke (width 0) (type default))
@@
     (stroke (width 0) (type default))
   )
+  (wire (pts (xy 34.29 144.145) (xy 48.26 144.145))
+    (stroke (width 0) (type default))
+  )
   (wire (pts (xy 257.81 109.22) (xy 257.81 107.95))
     (stroke (width 0) (type default))
@@
     (stroke (width 0) (type default))
   )
-  (wire (pts (xy 34.29 168.91) (xy 34.29 154.94))
-    (stroke (width 0) (type default))
-  )
   (wire (pts (xy 266.7 33.655) (xy 274.955 33.655))
     (stroke (width 0) (type default))
@@
     (stroke (width 0) (type default))
   )
-  (wire (pts (xy 48.26 168.91) (xy 34.29 168.91))
-    (stroke (width 0) (type default))
-  )
   (wire (pts (xy 116.84 96.52) (xy 119.38 96.52))
     (stroke (width 0) (type default))
@@
     (stroke (width 0) (type default))
   )
+  (wire (pts (xy 86.36 147.955) (xy 74.295 147.955))
+    (stroke (width 0) (type default))
+  )
   (wire (pts (xy 226.06 138.43) (xy 226.06 146.05))
     (stroke (width 0) (type default))
@@
     (stroke (width 0) (type default))
   )
+  (wire (pts (xy 36.195 157.48) (xy 36.195 168.91))
+    (stroke (width 0) (type default))
+  )
   (wire (pts (xy 146.05 99.06) (xy 147.32 99.06))
     (stroke (width 0) (type default))
@@
     (stroke (width 0) (type default))
   )
-  (wire (pts (xy 36.195 144.145) (xy 48.26 144.145))
-    (stroke (width 0) (type default))
-  )
   (wire (pts (xy 152.4 77.47) (xy 152.4 76.2))
     (stroke (width 0) (type default))
@@
   )
   (symbol (lib_id "power:GND") (at 68.58 139.065 0) (unit 1)
-    (in_bom yes) (on_board yes) (dnp no) (fields_autoplaced)
+    (in_bom yes) (on_board yes) (dnp no)
     (property "Reference" "#PWR057" (at 68.58 145.415 0)
       (effects (font (size 1.27 1.27)) hide)
     )
-    (property "Value" "GND" (at 68.58 144.145 0)
+    (property "Value" "GND" (at 71.755 141.605 0)
       (effects (font (size 1.27 1.27)))
     )
