File: V2/Hardware/Plantomation_V2.kicad_pcb (KiCad board)
At the start: 4 copper layers, 100 x 100 mm, 203 parts, among them J101 USB_B, J102 12V In, J201 Valves, J202 Pump1, J203 Pump2, J204 Shifter, J301 Sig, J302 Temp, J303 Vcc, J304 Air_Hue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

Commit message: prepare code and 3d files
Other:
- board text added: "JLCJLCJLCJLC"
